File: Placa De Ganho 2026.kicad_sch (KiCad schematic)
At the start: 40 parts, among them J1 Conn_Output, J2 Conn_01x01_Pin, J3 Conn_Sensores, J4 Conn_Alimentacao, U1 AD625JNZ, U2 AD625JNZ, U3 AD744JNZ, U4 AD744JNZ

Commit message: 11_07_2026
Parts:
- removed J1: Conn_Output, Connector_PinHeader_1.00mm:PinHeader_1x02_P1.00mm_Vertical, symbol Connector:Conn_01x02_Pin
- removed J3: Conn_Sensores, Connector_PinHeader_1.27mm:PinHeader_1x07_P1.27mm_Vertical, symbol Connector:Conn_01x07_Pin
- added J1: Conn_Estagio_3_Out, Connector_Pin:Pin_D1.0mm_L10.0mm, symbol Connector:Conn_01x01_Pin
- added J3: Conn_Wheatstone01, Cangaco:CANGACO_PinHeader_1x02_0.8mm, symbol Connector:Conn_01x02_Pin
- added J5: Conn_Wheatstone_02, Cangaco:CANGACO_PinHeader_1x02_0.8mm, symbol Connector:Conn_01x02_Pin
- added J6: Conn_Wheatstone_Alim, TerminalBlock_CUI:TerminalBlock_CUI_TB007-508-03_1x03_P5.08mm_Horizontal, symbol Connector:Conn_01x03_Pin
- added J7: Conn_Terra_Out, Connector_Pin:Pin_D1.0mm_L10.0mm, symbol Connector:Conn_01x01_Pin
- J2: value Conn_01x01_Pin -> Conn_Estagio_2_Out
- R1, R2, R3, R4, R5, R6, R7, R8, R9, Rf1, Rf2, Rf3, Rf4, Rg1, Rg2: footprint Resistor_THT:R_Axial_DIN0204_L3.6mm_D1.6mm_P5.08mm_Horizontal -> Cangaco:CANGACO_Resistor_0.8mm
- RV1, RV2, RV3: footprint Cangaço:SPACE-Potentiometer_Bourns_3296W_Vertical -> Cangaco:SPACE-Potentiometer_Bourns_3296W_Vertical
Connections:
- net GND: now also J6.2 (Pin_2), J7.1 (Pin_1)
- net VDD: now also J6.1 (Pin_1)
- net VSS: now also J6.3 (Pin_3)
- net at C14.1, R3.2, U4.6 (OUT): now also J1.1 (Pin_1)
- net at R6.1: now also J3.2 (Pin_2)
- net at R5.1: now also J3.1 (Pin_1)
- net at R7.1: now also J5.1 (Pin_1)
- net at R8.1: now also J5.2 (Pin_2)
